File: pcb/csi-analogvideo-capture.kicad_sch (KiCad schematic)
At the start: 67 parts

Commit message: update schematicand pcb, DRC passed
Parts:
- removed C? (x5): 0.1μF, symbol Device:C_Feedthrough
- removed H? (x4): MountingHole, MountingHole:MountingHole_3.2mm_M3_ISO14580, symbol Mechanical:MountingHole
- removed R? (x2): R, Resistor_SMD:R_0603_1608Metric_Pad1.05x0.95mm_HandSolder, symbol Device:R
- removed U?: TPS79901DDCR, Package_TO_SOT_SMD:SOT-23-5, symbol TPS79901DDCR:TPS79901DDCR
- added FB1, FB2, FB3, FB4, FB5: 600Ω, Inductor_SMD:L_0603_1608Metric, symbol Device:FerriteBead
- added TP1, TP2, TP3, TP4, TP5, TP6: TestPoint, TestPoint:TestPoint_Pad_D1.0mm, symbol Connector:TestPoint
- added U2: NJM12888F18, Package_TO_SOT_SMD:SOT-23-5, symbol NJM12888F18:NJM12888F18
- C1, C10, C11, C12, C16, C17, C18, C19, C2, C20, C21, C22, C23, C24, C25, C26, C27, C28, C29, C3, C30, C4, C5, C6, C7, C8, C9: renamed from C?; footprint Capacitor_SMD:C_0603_1608Metric_Pad1.05x0.95mm_HandSolder -> Capacitor_SMD:C_0402_1005Metric
- C13, C15: renamed from C?; footprint Capacitor_SMD:C_0603_1608Metric_Pad1.05x0.95mm_HandSolder -> Capacitor_SMD:C_1206_3216Metric
- C14: renamed from C?; value C -> 10nF; footprint Capacitor_SMD:C_0603_1608Metric_Pad1.05x0.95mm_HandSolder -> Capacitor_SMD:C_0402_1005Metric
- J1: renamed from J?; footprint (none) -> Connector_PinHeader_2.54mm:PinHeader_2x08_P2.54mm_Vertical
- J2: renamed from CN?; footprint (none) -> Connector_FFC-FPC:TE_1-84953-5_1x15-1MP_P1.0mm_Horizontal
- R1, R10, R11, R12, R13, R14, R15, R16, R17, R18, R19, R2, R20, R21, R3, R4, R5, R6, R7, R8, R9: renamed from R?; footprint Resistor_SMD:R_0603_1608Metric_Pad1.05x0.95mm_HandSolder -> Resistor_SMD:R_0402_1005Metric
- U1: renamed from U?; footprint (none) -> Package_CSP:LFCSP-32-1EP_5x5mm_P0.5mm_EP3.25x3.25mm
- Y1: renamed from Y?; footprint Crystal:Crystal_SMD_3225-4Pin_3.2x2.5mm_HandSoldering -> Crystal:Crystal_SMD_3225-4Pin_3.2x2.5mm
Connections:
- net +1V8: now also FB2.1, FB3.1, FB4.1, FB5.1, U2.5 (VOUT); no longer C14.1
- net +3V3: now also FB1.1, U2.1 (VIN), U2.3 (CTRL)
- net AVDD_1V8: now also FB3.2
- net DVDDIO_3V3: now also FB1.2
- net DVDD_1V8: now also FB2.2
- net GND: now also C14.2, U2.2 (GND)
- net MVDD_1V8: now also FB4.2
- net PVDD_1V8: now also FB5.2
- net ~{INTRQ}: now reaches U1.5 (~{INTRQ})
- net ~{INTRQ}: now also TP1.1
- net GPO2: now reaches U1.6 (GPO2)
- net GPO2: now also TP2.1
- net GPO1: now reaches U1.7 (GPO1)
- net GPO1: now also TP3.1
- net GPO0: now reaches U1.8 (GPO0)
- net GPO0: now also TP4.1
- net GPIO1: now reaches J2.4 (GPIO1)
- net GPIO1: now also TP6.1
- net GPIO0: now reaches J2.5 (GPIO0)
- net GPIO0: now also TP5.1
- new net: C14.1, U2.4 (CS)
- no-connect marks 4 -> 2
Other:
- note added: "1.0mm 15P ZIF upper contact"
- moved on the sheet: C13, C14, C15, J2

Commit message: clean up project, update pcb
Parts:
- J2: value rpi_camera_conn_top -> RPI_CSI_TOP; symbol rpi_camera_conn:rpi_camera_conn_top -> RPI_CSI_CONN:RPI_CSI_TOP
Other:
- note added: "ALSB High -> I2C Addr. 0x42 ALSB Low -> I2C Addr. 0x40"
- note added: "Use 1.0mm 15P upper contact ZIF connector e.g.) Wurth Elektronik 68611514122"
- note removed: "1.0mm 15P ZIF upper contact"
- note removed: "ALSB High: I2C Addr. 0x42 ALSB Low : I2C Addr. 0x40"
Changed lines of the file:
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@@
     (stroke (width 0) (type default) (color 0 0 0 0))
   )
-  (text "1.0mm 15P ZIF upper contact" (at 186.69 148.59 0)
-    (effects (font (size 1.27 1.27)) (justify left bottom))
-  )
-  (text "ALSB High: I2C Addr. 0x42\nALSB Low : I2C Addr. 0x40"
-    (at 226.06 195.58 0)
+  (text "Use 1.0mm 15P upper contact ZIF connector\ne.g.) Wurth Elektronik 68611514122"
+    (at 179.07 154.94 0)
+    (effects (font (size 1.27 1.27)) (justify left bottom))
+  )
+  (text "ALSB High -> I2C Addr. 0x42\nALSB Low -> I2C Addr. 0x40"
+    (at 144.78 170.18 0)
     (effects (font (size 1.27 1.27)) (justify left bottom))
   )
@@
     (pin "2")
   )
-  (symbol (lib_id "rpi_camera_conn:rpi_camera_conn_top") (at 184.15 121.92 0) (unit 1)
+  (symbol (lib_id "RPI_CSI_CONN:RPI_CSI_TOP") (at 184.15 121.92 0) (unit 1)
     (in_bom yes) (on_board yes) (fields_autoplaced)
     (property "Reference" "J2" (id 0) (at 190.5 120.6499 0)
       (effects (font (size 1.27 1.27)) (justify left))
     )
-    (property "Value" "rpi_camera_conn_top" (id 1) (at 190.5 123.1899 0)
+    (property "Value" "RPI_CSI_TOP" (id 1) (at 190.5 123.1899 0)
       (effects (font (size 1.27 1.27)) (justify left))
     )
@@
     )
     (path "/c5c5a7ba-cf68-466b-ab80-8f1be5bf9c84"
-      (reference "J2") (unit 1) (value "rpi_camera_conn_top") (footprint "Connector_FFC-FPC:TE_1-84953-5_1x15-1MP_P1.0mm_Horizontal")
+      (reference "J2") (unit 1) (value "RPI_CSI_TOP") (footprint "Connector_FFC-FPC:TE_1-84953-5_1x15-1MP_P1.0mm_Horizontal")
     )
     (path "/00000000-0000-0000-0000-00005bf19426"
