File: pcb/sdtv2csi.kicad_pcb (KiCad board)
At the start: 2 copper layers, 25 x 40 mm, 67 parts, among them J1 VIDEO_IN, J2 RPI_CSI_TOP, U1 ADV7280A-M, U2 NJM12888F18, Y1 ABM8G-28.63636MHZ

Commit message: pcb: migrate KiCad to 9.0.1
Other:
- board text added: "Thickness: 0.8mm Min Track/Spacing: 6/6mil Min Hole Size 0.3mm"
